File: pcb/interface/interface.kicad_pcb (KiCad board)
At the start: 4 copper layers, 49.2 x 49.2 mm, 20 parts, among them J1 Conn_ARM_JTAG_SWD_10, J4 Conn_01x05_Pin, J5 Conn_01x05_Pin, U1 MT6701CT

Commit message: docs update
Parts:
- J1: footprint kuleana:SAMTEC_FTSH-105-XX-X-DV -> Connector_PinHeader_1.27mm:PinHeader_2x05_P1.27mm_Vertical_SMD
- turned J1 to 180 degrees
