File: pcb/interface/interface.kicad_sch (KiCad schematic)
At the start: 20 parts, among them J1 Conn_ARM_JTAG_SWD_10, J4 Conn_01x05_Pin, J5 Conn_01x05_Pin, U1 MT6701CT

Commit message: docs update
Parts:
- J1: footprint kuleana:SAMTEC_FTSH-105-XX-X-DV -> Connector_PinHeader_1.27mm:PinHeader_2x05_P1.27mm_Vertical_SMD
Changed lines of the file:
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@@
 			)
 		)
-		(property "Footprint" "kuleana:SAMTEC_FTSH-105-XX-X-DV"
+		(property "Footprint" "Connector_PinHeader_1.27mm:PinHeader_2x05_P1.27mm_Vertical_SMD"
 			(at 40.64 127 0)
 			(hide yes)
